File: czujnikParkowania.sch (KiCad schematic (older format))
At the start: 38 parts, among them J1 Screw_Terminal_01x03, Q1 BC817, Q2 IRF7404, Q3 BC817, Q4 BC817, Q5 BC817, U1 DC56-11SEKWA, U2 LM7805_TO220, U3 HC-SR04

Commit message: added caps and button
Parts:
- added C10, C7, C8, C9: 100n, Capacitor_SMD:C_0805_2012Metric, symbol Device:C
- added SW1: SW_Push, Button_Switch_SMD:SW_SPST_B3S-1000, symbol Switch:SW_Push
Connections:
- net +5V: now also C10.1, C7.1, C8.1, C9.1
- net GND: now also C10.2, C7.2, C8.2, C9.2, SW1.2
- net BTN: now reaches A1.1 (D1/TX)
- net BTN: now also SW1.1
- no-connect marks 14 -> 13
Changed lines of the file:
@@
 NoConn ~ 3300 3000
 NoConn ~ 3300 3100
-NoConn ~ 2300 1900
 Wire Wire Line
 	2300 1800 1800 1800
@@
 L power:+5V #PWR0121
 U 1 1 5EB28EBD
-P 6850 5150
-F 0 "#PWR0121" H 6850 5000 50  0001 C CNN
-F 1 "+5V" H 6865 5323 50  0000 C CNN
-F 2 "" H 6850 5150 50  0001 C CNN
-F 3 "" H 6850 5150 50  0001 C CNN
-	1    6850 5150
+P 6850 4950
+F 0 "#PWR0121" H 6850 4800 50  0001 C CNN
+F 1 "+5V" H 6865 5123 50  0000 C CNN
+F 2 "" H 6850 4950 50  0001 C CNN
+F 3 "" H 6850 4950 50  0001 C CNN
+	1    6850 4950
 	1    0    0    -1
 $EndComp
@@
 L power:+5V #PWR0122
 U 1 1 5EB296B5
-P 7650 5150
-F 0 "#PWR0122" H 7650 5000 50  0001 C CNN
-F 1 "+5V" H 7665 5323 50  0000 C CNN
-F 2 "" H 7650 5150 50  0001 C CNN
-F 3 "" H 7650 5150 50  0001 C CNN
-	1    7650 5150
+P 7650 4950
+F 0 "#PWR0122" H 7650 4800 50  0001 C CNN
+F 1 "+5V" H 7665 5123 50  0000 C CNN
+F 2 "" H 7650 4950 50  0001 C CNN
+F 3 "" H 7650 4950 50  0001 C CNN
+	1    7650 4950
 	1    0    0    -1
 $EndComp
@@
 L power:+5V #PWR0123
 U 1 1 5EB2995A
-P 8450 5150
-F 0 "#PWR0123" H 8450 5000 50  0001 C CNN
-F 1 "+5V" H 8465 5323 50  0000 C CNN
-F 2 "" H 8450 5150 50  0001 C CNN
-F 3 "" H 8450 5150 50  0001 C CNN
-	1    8450 5150
+P 8450 4950
+F 0 "#PWR0123" H 8450 4800 50  0001 C CNN
+F 1 "+5V" H 8465 5123 50  0000 C CNN
+F 2 "" H 8450 4950 50  0001 C CNN
+F 3 "" H 8450 4950 50  0001 C CNN
+	1    8450 4950
 	1    0    0    -1
 $EndComp
@@
 L power:+5V #PWR0124
 U 1 1 5EB29CCE
-P 9250 5150
-F 0 "#PWR0124" H 9250 5000 50  0001 C CNN
-F 1 "+5V" H 9265 5323 50  0000 C CNN
-F 2 "" H 9250 5150 50  0001 C CNN
-F 3 "" H 9250 5150 50  0001 C CNN
-	1    9250 5150
-	1    0    0    -1
-$EndComp
-Wire Wire Line
-	6850 5150 6850 5300
-Wire Wire Line
-	7650 5150 7650 5300
-Wire Wire Line
-	8450 5150 8450 5300
-Wire Wire Line
-	9250 5150 9250 5300
+P 9250 4950
+F 0 "#PWR0124" H 9250 4800 50  0001 C CNN
+F 1 "+5V" H 9265 5123 50  0000 C CNN
+F 2 "" H 9250 4950 50  0001 C CNN
+F 3 "" H 9250 4950 50  0001 C CNN
+	1    9250 4950
+	1    0    0    -1
+$EndComp
 Wire Wire Line
 	6350 5600 6550 5600
@@
 Text GLabel 1150 6150 0    50   Input ~ 0
 R
+$Comp
+L Switch:SW_Push SW1
+U 1 1 5EABA31B
+P 4200 3800
+F 0 "SW1" H 4200 4085 50  0000 C CNN
+F 1 "SW_Push" H 4200 3994 50  0000 C CNN
+F 2 "Button_Switch_SMD:SW_SPST_B3S-1000" H 4200 4000 50  0001 C CNN
+F 3 "https://www.tme.eu/pl/details/b3s-1000/mikroprzelaczniki-tact/omron-ocb/" H 4200 4000 50  0001 C CNN
+	1    4200 3800
+	1    0    0    -1
+$EndComp
+$Comp
+L power:GND #PWR0125
+U 1 1 5EABA92C
+P 4700 3950
+F 0 "#PWR0125" H 4700 3700 50  0001 C CNN
+F 1 "GND" H 4705 3777 50  0000 C CNN
+F 2 "" H 4700 3950 50  0001 C CNN
+F 3 "" H 4700 3950 50  0001 C CNN
+	1    4700 3950
+	1    0    0    -1
+$EndComp
+Wire Wire Line
+	4400 3800 4700 3800
+Wire Wire Line
+	4700 3800 4700 3950
+Wire Wire Line
+	4000 3800 3650 3800
+Wire Wire Line
+	2300 1900 1800 1900
+Text Label 1800 1900 0    50   ~ 0
+BTN
+Text Label 3650 3800 0    50   ~ 0
+BTN
+Wire Wire Line
+	9250 4950 9250 5100
+Wire Wire Line
+	8450 4950 8450 5100
+Wire Wire Line
+	7650 4950 7650 5100
+Wire Wire Line
+	6850 4950 6850 5100
+$Comp
+L Device:C C7
+U 1 1 5EBDFF34
+P 6600 5100
+F 0 "C7" V 6348 5100 50  0000 C CNN
+F 1 "100n" V 6439 5100 50  0000 C CNN
+F 2 "Capacitor_SMD:C_0805_2012Metric" H 6638 4950 50  0001 C CNN
+F 3 "~" H 6600 5100 50  0001 C CNN
+	1    6600 5100
+	0    1    1    0
+$EndComp
+$Comp
+L Device:C C8
+U 1 1 5EBE0407
+P 7400 5100
+F 0 "C8" V 7148 5100 50  0000 C CNN
+F 1 "100n" V 7239 5100 50  0000 C CNN
+F 2 "Capacitor_SMD:C_0805_2012Metric" H 7438 4950 50  0001 C CNN
+F 3 "~" H 7400 5100 50  0001 C CNN
+	1    7400 5100
+	0    1    1    0
+$EndComp
+$Comp
+L Device:C C9
+U 1 1 5EBE090B
+P 8200 5100
+F 0 "C9" V 7948 5100 50  0000 C CNN
+F 1 "100n" V 8039 5100 50  0000 C CNN
+F 2 "Capacitor_SMD:C_0805_2012Metric" H 8238 4950 50  0001 C CNN
+F 3 "~" H 8200 5100 50  0001 C CNN
+	1    8200 5100
+	0    1    1    0
+$EndComp
+$Comp
+L Device:C C10
+U 1 1 5EBE0DA2
+P 9000 5100
+F 0 "C10" V 8748 5100 50  0000 C CNN
+F 1 "100n" V 8839 5100 50  0000 C CNN
+F 2 "Capacitor_SMD:C_0805_2012Metric" H 9038 4950 50  0001 C CNN
+F 3 "~" H 9000 5100 50  0001 C CNN
+	1    9000 5100
+	0    1    1    0
+$EndComp
+$Comp
+L power:GND #PWR0126
+U 1 1 5EBE1987
+P 6350 5150
+F 0 "#PWR0126" H 6350 4900 50  0001 C CNN
+F 1 "GND" H 6355 4977 50  0000 C CNN
+F 2 "" H 6350 5150 50  0001 C CNN
+F 3 "" H 6350 5150 50  0001 C CNN
+	1    6350 5150
+	1    0    0    -1
+$EndComp
+$Comp
+L power:GND #PWR0127
+U 1 1 5EBE1CC0
+P 7150 5150
+F 0 "#PWR0127" H 7150 4900 50  0001 C CNN
+F 1 "GND" H 7155 4977 50  0000 C CNN
+F 2 "" H 7150 5150 50  0001 C CNN
+F 3 "" H 7150 5150 50  0001 C CNN
+	1    7150 5150
+	1    0    0    -1
+$EndComp
+$Comp
+L power:GND #PWR0128
+U 1 1 5EBE1F68
+P 7950 5150
+F 0 "#PWR0128" H 7950 4900 50  0001 C CNN
+F 1 "GND" H 7955 4977 50  0000 C CNN
+F 2 "" H 7950 5150 50  0001 C CNN
+F 3 "" H 7950 5150 50  0001 C CNN
+	1    7950 5150
+	1    0    0    -1
+$EndComp
+$Comp
+L power:GND #PWR0129
+U 1 1 5EBE225E
+P 8750 5150
+F 0 "#PWR0129" H 8750 4900 50  0001 C CNN
+F 1 "GND" H 8755 4977 50  0000 C CNN
+F 2 "" H 8750 5150 50  0001 C CNN
+F 3 "" H 8750 5150 50  0001 C CNN
+	1    8750 5150
+	1    0    0    -1
+$EndComp
+Wire Wire Line
+	9150 5100 9250 5100
+Connection ~ 9250 5100
+Wire Wire Line
+	9250 5100 9250 5300
+Wire Wire Line
+	8850 5100 8750 5100
+Wire Wire Line
+	8750 5100 8750 5150
+Wire Wire Line
+	8050 5100 7950 5100
+Wire Wire Line
+	7950 5100 7950 5150
+Wire Wire Line
+	7250 5100 7150 5100
+Wire Wire Line
+	7150 5100 7150 5150
+Wire Wire Line
+	7550 5100 7650 5100
+Connection ~ 7650 5100
+Wire Wire Line
+	7650 5100 7650 5300
+Wire Wire Line
+	8350 5100 8450 5100
+Connection ~ 8450 5100
+Wire Wire Line
+	8450 5100 8450 5300
+Wire Wire Line
+	6750 5100 6850 5100
+Connection ~ 6850 5100
+Wire Wire Line
+	6850 5100 6850 5300
+Wire Wire Line
+	6450 5100 6350 5100
+Wire Wire Line
+	6350 5100 6350 5150
 $EndSCHEMATC

Commit message: added GND plane on back
Parts:
- added C11, C12, C13: 100n, Capacitor_SMD:C_0805_2012Metric, symbol Device:C
- added R15: 1k, Resistor_SMD:R_0805_2012Metric, symbol Device:R
- added U4: ATmega328-AU, Package_QFP:TQFP-32_7x7mm_P0.8mm, symbol MCU_Microchip_ATmega:ATmega328-AU
- added Y1: Crystal, MYCONN:16MHz cristal oscillator, symbol Device:Crystal
- C5: value 100n -> 10n
- C8, C9: value 100n -> 1p
- R4: value 10k -> 1k
Connections:
- net +5V: now also C11.1, C12.1, C13.1, R15.1, U4.18 (AVCC), U4.4 (VCC), U4.6 (VCC); no longer A1.18 (AREF), C7.1, C8.1, C9.1, R4.1
- net BTN: now also U4.31 (PD1)
- net BUZZER: now also U4.17 (PB5)
- net ECHO: now also U4.13 (PB1)
- net GND: now also C8.1, C9.1, R4.2, C11.2, C12.2, C13.2, U4.21 (GND), U4.3 (GND), U4.5 (GND); no longer C8.2, C9.2
- net RGB_DI: now also U4.30 (PD0)
- net SEG_1: now also U4.15 (PB3)
- net SEG_2: now also U4.16 (PB4)
- net SEG_A: now also U4.32 (PD2)
- net SEG_B: now also U4.1 (PD3)
- net SEG_C: now also U4.2 (PD4)
- net SEG_D: now also U4.9 (PD5)
- net SEG_E: now also U4.10 (PD6)
- net SEG_F: now also U4.11 (PD7)
- net SEG_G: now also U4.12 (PB0)
- net TRIG: now also U4.14 (PB2)
- net at A1.28 (~RESET), A1.3 (~RESET): now also R15.2; no longer R4.2
- new net: A1.18 (AREF), C7.1, U4.20 (AREF)
- new net: R4.1, U4.29 (~RESET~/PC6)
- new net: C8.2, U4.7 (XTAL1/PB6), Y1.1
- new net: C9.2, U4.8 (XTAL2/PB7), Y1.2
- no-connect marks 13 -> 21
Other:
- moved on the sheet: BZ1, C1, C2, C3, C4, C5, C6, D1, D2, D3, D4, D5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

Commit message: added GND plane on back. wrong brd in prev upload
Parts:
- removed C11, C12, C13: 100n, Capacitor_SMD:C_0805_2012Metric, symbol Device:C
- removed R15: 1k, Resistor_SMD:R_0805_2012Metric, symbol Device:R
- removed U4: ATmega328-AU, Package_QFP:TQFP-32_7x7mm_P0.8mm, symbol MCU_Microchip_ATmega:ATmega328-AU
- removed Y1: Crystal, MYCONN:16MHz cristal oscillator, symbol Device:Crystal
- C5: value 10n -> 100n
- C8, C9: value 1p -> 100n
- R4: value 1k -> 10k
Connections:
- net +5V: now also A1.18 (AREF), C7.1, C8.1, C9.1, R4.1
- net GND: now also C8.2, C9.2; no longer C8.1, C9.1, R4.2
- net at A1.28 (~RESET), A1.3 (~RESET): now also R4.2
- no-connect marks 21 -> 13
Other:
- moved on the sheet: BZ1, C1, C2, C3, C4, C5, C6, D1, D2, D3, D4, D5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
